File: NixieClock.kicad_sch (KiCad schematic)
At the start: 0 parts

Commit message: Created shcema
Parts:
- added BT1: Battery_Cell, symbol Device:Battery_Cell
- added J_12V: Conn_01x02_Pin, Connector_PinHeader_2.00mm:PinHeader_1x02_P2.00mm_Vertical, symbol Connector:Conn_01x02_Pin
- added J_170V: Conn_01x01_Pin, Connector_PinHeader_2.00mm:PinHeader_1x01_P2.00mm_Vertical, symbol Connector:Conn_01x01_Pin
- added N1, N2, N3, N4: ~, NixieClock:Z570M, symbol NixieClock:Z570M
- added Q1_0, Q1_1, Q1_2, Q1_3, Q1_4, Q1_5, Q1_6, Q1_7, Q1_8, Q1_9, Q2_0, Q2_1, Q2_2, Q2_3, Q2_4, Q2_5, Q2_6, Q2_7, Q2_8, Q2_9, Q3_0, Q3_1, Q3_2, Q3_3, Q3_4, Q3_5, Q3_6, Q3_7, Q3_8, Q3_9, Q4_0, Q4_1, Q4_2, Q4_3, Q4_4, Q4_5, Q4_6, Q4_7, Q4_8, Q4_9: BC807, Package_TO_SOT_SMD:SOT-23_Handsoldering, symbol Transistor_BJT:BC807
- added R1_0, R1_1, R1_2, R1_3, R1_4, R1_5, R1_6, R1_7, R1_8, R1_9, R1_S, R2_0, R2_1, R2_2, R2_3, R2_4, R2_5, R2_6, R2_7, R2_8, R2_9, R2_S, R3_0, R3_1, R3_2, R3_3, R3_4, R3_5, R3_6, R3_7, R3_8, R3_9, R3_S, R4_0, R4_1, R4_2, R4_3, R4_4, R4_5, R4_6, R4_7, R4_8, R4_9, R4_S: R, Resistor_SMD:R_1206_3216Metric_Pad1.30x1.75mm_HandSolder, symbol Device:R
- added REG1: LF50_TO252, Package_TO_SOT_SMD:TO-252-2, symbol Regulator_Linear:LF50_TO252
- added RTC1: DS1307+, Package_DIP:DIP-8_W7.62mm_SMDSocket_SmallPads, symbol Timer_RTC:DS1307+
- added SR1, SR2, SR3, SR4, SR5: HEF4094BT, SOT109-1_NXP, symbol NixieClock:HEF4094BT
- added U1: ATtiny24A-SS, Package_SO:SOIC-14_3.9x8.7mm_P1.27mm, symbol MCU_Microchip_ATtiny:ATtiny24A-SS
Connections:
- new net: N2.1, Q2_1.3 (C)
- new net: N2.11 (9), Q2_9.3 (C)
- new net: N2.12 (0), Q2_0.3 (C)
- new net: N2.13 (A), R2_S.1
- new net: N2.2, Q2_2.3 (C)
- new net: N2.3, Q2_3.3 (C)
- new net: N2.5 (4), Q2_4.3 (C)
- new net: N2.6 (5), Q2_5.3 (C)
- new net: N2.7 (6), Q2_6.3 (C)
- new net: N2.8 (7), Q2_7.3 (C)
- new net: N2.9 (8), Q2_8.3 (C)
- new net: R4_2.1, SR5.4 (QP0)
- new net: Q4_2.1 (B), R4_2.2
- new net: R4_1.1, SR4.11 (QP7)
- new net: Q4_1.1 (B), R4_1.2
- new net: BT1.2 (-), J_12V.1 (Pin_1), Q1_0.2 (E), Q1_1.2 (E), Q1_2.2 (E), Q1_3.2 (E), Q1_4.2 (E), Q1_5.2 (E), Q1_6.2 (E), Q1_7.2 (E), Q1_8.2 (E), Q1_9.2 (E), Q2_0.2 (E), Q2_1.2 (E), Q2_2.2 (E), Q2_3.2 (E), Q2_4.2 (E), Q2_5.2 (E), Q2_6.2 (E), Q2_7.2 (E), Q2_8.2 (E), Q2_9.2 (E), Q3_0.2 (E), Q3_1.2 (E), Q3_2.2 (E), Q3_3.2 (E), Q3_4.2 (E), Q3_5.2 (E), Q3_6.2 (E), Q3_7.2 (E), Q3_8.2 (E), Q3_9.2 (E), Q4_0.2 (E), Q4_1.2 (E), Q4_2.2 (E), Q4_3.2 (E), Q4_4.2 (E), Q4_5.2 (E), Q4_6.2 (E), Q4_7.2 (E), Q4_8.2 (E), Q4_9.2 (E), REG1.2 (GND), RTC1.4 (GND), SR1.8 (VSS), SR2.8 (VSS), SR3.8 (VSS), SR4.8 (VSS), SR5.8 (VSS)
- new net: N4.2, Q4_2.3 (C)
- new net: Q4_3.1 (B), R4_3.2
- new net: N4.3, Q4_3.3 (C)
- new net: R2_2.1, SR2.14 (QP4)
- new net: Q2_2.1 (B), R2_2.2
- new net: Q1_7.1 (B), R1_7.2
- new net: N1.8 (7), Q1_7.3 (C)
- new net: Q2_8.1 (B), R2_8.2
- new net: R4_7.1, SR5.13 (QP5)
- new net: Q4_7.1 (B), R4_7.2
- new net: R1_6.1, SR1.12 (QP6)
- new net: Q1_6.1 (B), R1_6.2
- new net: R2_6.1, SR3.4 (QP0)
- new net: Q2_6.1 (B), R2_6.2
- new net: R1_0.1, SR1.4 (QP0)
- new net: Q1_0.1 (B), R1_0.2
- new net: Q1_4.1 (B), R1_4.2
- new net: N1.5 (4), Q1_4.3 (C)
- new net: N3.1, Q3_1.3 (C)
- new net: N3.11 (9), Q3_9.3 (C)
- new net: N3.12 (0), Q3_0.3 (C)
- new net: N3.13 (A), R3_S.1
- new net: N3.2, Q3_2.3 (C)
- new net: N3.3, Q3_3.3 (C)
- new net: N3.5 (4), Q3_4.3 (C)
- new net: N3.6 (5), Q3_5.3 (C)
- new net: N3.7 (6), Q3_6.3 (C)
- new net: N3.8 (7), Q3_7.3 (C)
- new net: N3.9 (8), Q3_8.3 (C)
- new net: Q2_9.1 (B), R2_9.2
- new net: Q3_0.1 (B), R3_0.2
- new net: R2_7.1, SR3.5 (QP1)
- new net: Q2_7.1 (B), R2_7.2
- new net: Q4_8.1 (B), R4_8.2
- new net: N4.9 (8), Q4_8.3 (C)
- new net: Q2_4.1 (B), R2_4.2
- new net: Q3_1.1 (B), R3_1.2
- new net: R2_5.1, SR2.11 (QP7)
- new net: Q2_5.1 (B), R2_5.2
- new net: R4_5.1, SR5.7 (QP3)
- new net: Q4_5.1 (B), R4_5.2
- new net: J_12V.2 (Pin_2), REG1.1 (VI)
- new net: REG1.3 (VO), RTC1.8 (VCC), SR1.16 (VDD), SR2.16 (VDD), SR3.16 (VDD), SR4.16 (VDD), SR5.16 (VDD)
- new net: SR1.1 (STR), SR2.1 (STR), SR3.1 (STR), SR4.1 (STR), SR5.1 (STR)
- new net: R4_9.1, SR5.11 (QP7)
- new net: R4_8.1, SR5.12 (QP6)
- new net: R4_6.1, SR5.14 (QP4)
- new net: SR4.9 (QS1), SR5.2 (D)
- new net: SR1.3 (CP), SR2.3 (CP), SR3.3 (CP), SR4.3 (CP), SR5.3 (CP)
- new net: R4_3.1, SR5.5 (QP1)
- new net: R4_4.1, SR5.6 (QP2)
- new net: Q4_0.1 (B), R4_0.2
- new net: N4.12 (0), Q4_0.3 (C)
- new net: Q3_9.1 (B), R3_9.2
- new net: R1_9.1, SR2.5 (QP1)
- new net: Q1_9.1 (B), R1_9.2
- new net: R1_1.1, SR1.5 (QP1)
- new net: Q1_1.1 (B), R1_1.2
- new net: Q3_3.1 (B), R3_3.2
- new net: Q4_6.1 (B), R4_6.2
- new net: N4.7 (6), Q4_6.3 (C)
- new net: R2_9.1, SR3.7 (QP3)
- new net: N1.7 (6), Q1_6.3 (C)
- new net: N1.1, Q1_1.3 (C)
- new net: N1.11 (9), Q1_9.3 (C)
- new net: N1.12 (0), Q1_0.3 (C)
- new net: N1.13 (A), R1_S.1
- new net: N1.2, Q1_2.3 (C)
- new net: N1.3, Q1_3.3 (C)
- new net: N1.6 (5), Q1_5.3 (C)
- new net: N1.9 (8), Q1_8.3 (C)
- new net: Q4_9.1 (B), R4_9.2
- new net: N4.11 (9), Q4_9.3 (C)
- new net: R3_7.1, SR4.7 (QP3)
- new net: Q3_7.1 (B), R3_7.2
- new net: R3_3.1, SR3.11 (QP7)
- new net: R3_2.1, SR3.12 (QP6)
- new net: R3_1.1, SR3.13 (QP5)
- new net: R3_0.1, SR3.14 (QP4)
- new net: SR2.9 (QS1), SR3.2 (D)
- new net: R2_8.1, SR3.6 (QP2)
- new net: SR3.9 (QS1), SR4.2 (D)
- new net: Q1_2.1 (B), R1_2.2
- new net: R3_8.1, SR4.14 (QP4)
- new net: Q3_8.1 (B), R3_8.2
- new net: J_170V.1 (Pin_1), R1_S.2, R2_S.2, R3_S.2, R4_S.2
- new net: BT1.1 (+), RTC1.3 (VBAT)
- new net: Q2_3.1 (B), R2_3.2
- new net: R2_0.1, SR2.6 (QP2)
- new net: Q2_0.1 (B), R2_0.2
- new net: R2_1.1, SR2.7 (QP3)
- new net: Q2_1.1 (B), R2_1.2
- new net: R1_4.1, SR1.14 (QP4)
- new net: R1_7.1, SR1.11 (QP7)
- new net: Q1_3.1 (B), R1_3.2
- new net: R1_5.1, SR1.13 (QP5)
- new net: Q1_5.1 (B), R1_5.2
- new net: R2_4.1, SR2.12 (QP6)
- new net: Q3_2.1 (B), R3_2.2
- new net: N4.8 (7), Q4_7.3 (C)
- new net: R3_9.1, SR4.13 (QP5)
- new net: Q3_6.1 (B), R3_6.2
- new net: R2_3.1, SR2.13 (QP5)
- new net: SR1.9 (QS1), SR2.2 (D)
- new net: R1_8.1, SR2.4 (QP0)
- new net: N4.1, Q4_1.3 (C)
- new net: N4.13 (A), R4_S.1
- new net: N4.5 (4), Q4_4.3 (C)
- new net: N4.6 (5), Q4_5.3 (C)
- new net: R1_2.1, SR1.6 (QP2)
- new net: Q3_4.1 (B), R3_4.2
- new net: R1_3.1, SR1.7 (QP3)
- new net: R4_0.1, SR4.12 (QP6)
- new net: R3_5.1, SR4.5 (QP1)
- new net: Q3_5.1 (B), R3_5.2
- new net: Q1_8.1 (B), R1_8.2
- new net: R3_4.1, SR4.4 (QP0)
- new net: R3_6.1, SR4.6 (QP2)
- new net: Q4_4.1 (B), R4_4.2

Commit message: update
Parts:
- added F1: Fuse, NixieClock:Breaker_Holder_5x20, symbol Device:Fuse
- added Y1: AB38T-32.768KHZ, AB38T-32.768KHZ:XTAL_AB38T-32.768KHZ, symbol NixieClock:AB38T-32.768KHZ
- added Y2: 16MHz, Crystal:Crystal_HC49-U_Vertical, symbol Device:Crystal
- renumbered U1 to MCU1
Connections:
- net GND: now reaches BT1.2 (-), J_12V.1 (Pin_1), Q1_0.2 (E), Q1_1.2 (E), Q1_2.2 (E), Q1_3.2 (E), Q1_4.2 (E), Q1_5.2 (E), Q1_6.2 (E), Q1_7.2 (E), Q1_8.2 (E), Q1_9.2 (E), Q2_0.2 (E), Q2_1.2 (E), Q2_2.2 (E), Q2_3.2 (E), Q2_4.2 (E), Q2_5.2 (E), Q2_6.2 (E), Q2_7.2 (E), Q2_8.2 (E), Q2_9.2 (E), Q3_0.2 (E), Q3_1.2 (E), Q3_2.2 (E), Q3_3.2 (E), Q3_4.2 (E), Q3_5.2 (E), Q3_6.2 (E), Q3_7.2 (E), Q3_8.2 (E), Q3_9.2 (E), Q4_0.2 (E), Q4_1.2 (E), Q4_2.2 (E), Q4_3.2 (E), Q4_4.2 (E), Q4_5.2 (E), Q4_6.2 (E), Q4_7.2 (E), Q4_8.2 (E), Q4_9.2 (E), REG1.2 (GND), RTC1.4 (GND), SR1.8 (VSS), SR2.8 (VSS), SR3.8 (VSS), SR4.8 (VSS), SR5.8 (VSS)
- net GND: now also MCU1.14 (GND), SR1.10 (QS2), SR2.10 (QS2), SR3.10 (QS2), SR4.10 (QS2), SR5.10 (QS2), SR5.9 (QS1)
- net +5V: now reaches MCU1.1 (VCC)
- net +5V: now also REG1.3 (VO), RTC1.8 (VCC), SR1.16 (VDD), SR2.16 (VDD), SR3.16 (VDD), SR4.16 (VDD), SR5.16 (VDD)
- net +12V: now reaches J_12V.2 (Pin_2), REG1.1 (VI)
- net STR: now reaches SR1.1 (STR), SR2.1 (STR), SR3.1 (STR), SR4.1 (STR), SR5.1 (STR)
- net OE: now reaches SR5.15 (OE)
- net OE: now also SR1.15 (OE), SR2.15 (OE), SR3.15 (OE), SR4.15 (OE)
- net CP: now reaches SR1.3 (CP), SR2.3 (CP), SR3.3 (CP), SR4.3 (CP), SR5.3 (CP)
- net +170V: now reaches J_170V.1 (Pin_1), R1_S.2, R2_S.2, R3_S.2, R4_S.2
- net +170V: now also F1.1, F1.2
- net at RTC1.1 (X1): now also Y1.1
- net at RTC1.2 (X2): now also Y1.2
Other:
- moved on the sheet: J_170V, MCU1

Commit message: updated schematic
Parts:
- removed Y1: AB38T-32.768KHZ, AB38T-32.768KHZ:XTAL_AB38T-32.768KHZ, symbol NixieClock:AB38T-32.768KHZ
- added CR1: 32,768KHz, symbol Device:Crystal
- added J_BTN: Conn_01x03_Pin, Connector_PinHeader_2.00mm:PinHeader_1x03_P2.00mm_Vertical, symbol Connector:Conn_01x03_Pin
- added J_DBG: Conn_01x04_Pin, Connector_PinHeader_2.00mm:PinHeader_1x04_P2.00mm_Vertical, symbol Connector:Conn_01x04_Pin
- BT1: value Battery_Cell -> CR2032; footprint (none) -> NixieClock:CR20_holder
- CR2: renamed from Y2; value 16MHz -> 10MHz; footprint Crystal:Crystal_HC49-U_Vertical -> Crystal:Crystal_SMD_HC49-SD_HandSoldering
- F1: value Fuse -> 250V/0.5A
- N1, N2, N3, N4: value ~ -> Z570M
- R1_0, R1_1, R1_2, R1_3, R1_4, R1_5, R1_6, R1_7, R1_8, R1_9, R2_0, R2_1, R2_2, R2_3, R2_4, R2_5, R2_6, R2_7, R2_8, R2_9, R3_0, R3_1, R3_2, R3_3, R3_4, R3_5, R3_6, R3_7, R3_8, R3_9, R4_0, R4_1, R4_2, R4_3, R4_4, R4_5, R4_6, R4_7, R4_8, R4_9: value R -> 5K1
- REG1: value LF50_TO252 -> LF50CDT-TR
- RS1: renamed from R1_S; value R -> 82K
- RS2: renamed from R2_S; value R -> 82K
- RS3: renamed from R3_S; value R -> 82K
- RS4: renamed from R4_S; value R -> 82K
Connections:
- net CP: now also MCU1.8 (PA5), J_DBG.2 (Pin_2)
- net GND: now also J_BTN.3 (Pin_3)
- net OE: now also MCU1.10 (PA3), J_DBG.4 (Pin_4)
- net STR: now also MCU1.11 (PA2), J_DBG.3 (Pin_3)
- net at MCU1.12 (PA1): now also J_BTN.1 (Pin_1)
- net at MCU1.13 (AREF/PA0): now also J_BTN.2 (Pin_2)
- net at MCU1.2 (XTAL1/PB0): now also CR2.1
- net at MCU1.6 (PA7): now also SR1.2 (D), J_DBG.1 (Pin_1)
- net at MCU1.7 (PA6): now also RTC1.5 (SDA)
- net at MCU1.9 (PA4): now also RTC1.6 (SCL)
- net at RTC1.1 (X1): now also CR1.1
- net at RTC1.2 (X2): now also CR1.2
Other:
- moved on the sheet: CR2, MCU1, SR5

Commit message: finished schematic
Parts:
- added C1: 1pF, Capacitor_SMD:C_1206_3216Metric_Pad1.33x1.80mm_HandSolder, symbol Device:C
- added C2: 2.2pF, Capacitor_SMD:C_1206_3216Metric_Pad1.33x1.80mm_HandSolder, symbol Device:C
- added R_PUP_RES1, R_PUP_SCL1, R_PUP_SDA1: 5K1, Resistor_SMD:R_1206_3216Metric_Pad1.30x1.75mm_HandSolder, symbol Device:R
- added SW_RES1: SW_Push, NixieClock:SW_TS1107GS, symbol Switch:SW_Push
Connections:
- net OE is gone; now on net CP: J_DBG.4 (Pin_4), MCU1.10 (PA3), SR1.15 (OE), SR2.15 (OE), SR3.15 (OE), SR4.15 (OE), SR5.15 (OE)
- net +5V: now also R_PUP_RES1.1, R_PUP_SCL1.1, R_PUP_SDA1.1
- net GND: now also C1.1, C2.1, SW_RES1.2
- net at CR2.1, MCU1.2 (XTAL1/PB0): now also C1.2
- net at MCU1.3 (XTAL2/PB1): now also CR2.2, C2.2
- net at MCU1.4 (~{RESET}/PB3): now also R_PUP_RES1.2, SW_RES1.1
- net at MCU1.7 (PA6), RTC1.5 (SDA): now also R_PUP_SDA1.2
- net at MCU1.9 (PA4), RTC1.6 (SCL): now also R_PUP_SCL1.2
Other:
- moved on the sheet: CR2, MCU1

Commit message: changes
Parts:
- CR1: footprint (none) -> NixieClock:XTAL_AB38T-32.768KHZ
- SR1, SR2, SR3, SR4, SR5: footprint SOT109-1_NXP -> NixieClock:SOT109-1_NXP-M
- renumbered J_12V to J_12V1, J_170V to J_170V1, J_BTN to J_BTN1, J_DBG to J_DBG1
Connections:
- net CP: no longer J_DBG1.4 (Pin_4), MCU1.10 (PA3), SR1.15 (OE), SR2.15 (OE), SR3.15 (OE), SR4.15 (OE), SR5.15 (OE)
- new net OE: J_DBG1.4 (Pin_4), MCU1.10 (PA3), SR1.15 (OE), SR2.15 (OE), SR3.15 (OE), SR4.15 (OE), SR5.15 (OE)
- no-connect marks 0 -> 10

Commit message: update
Parts:
- removed C1: 1pF, Capacitor_SMD:C_1206_3216Metric_Pad1.33x1.80mm_HandSolder, symbol Device:C
- removed C2: 2.2pF, Capacitor_SMD:C_1206_3216Metric_Pad1.33x1.80mm_HandSolder, symbol Device:C
- removed CR2: 10MHz, Crystal:Crystal_SMD_HC49-SD_HandSoldering, symbol Device:Crystal
- removed F1: 250V/0.5A, NixieClock:Breaker_Holder_5x20, symbol Device:Fuse
- added J_5V1, J_DBG_I2C1: Conn_01x02_Pin, Connector_PinHeader_2.54mm:PinHeader_1x02_P2.54mm_Vertical, symbol Connector:Conn_01x02_Pin
- added LED1, LED2: LED, LED_SMD:LED_1206_3216Metric_Pad1.42x1.75mm_HandSolder, symbol Device:LED
- added RL1: 200, Resistor_SMD:R_1206_3216Metric_Pad1.30x1.75mm_HandSolder, symbol Device:R
- J_12V1: footprint Connector_PinHeader_2.00mm:PinHeader_1x02_P2.00mm_Vertical -> Connector_PinHeader_2.54mm:PinHeader_1x02_P2.54mm_Vertical
- J_170V1: footprint Connector_PinHeader_2.00mm:PinHeader_1x01_P2.00mm_Vertical -> Connector_PinHeader_2.54mm:PinHeader_1x01_P2.54mm_Vertical
- J_BTN1: footprint Connector_PinHeader_2.00mm:PinHeader_1x03_P2.00mm_Vertical -> Connector_PinHeader_2.54mm:PinHeader_1x03_P2.54mm_Vertical
- J_DBG1: footprint Connector_PinHeader_2.00mm:PinHeader_1x04_P2.00mm_Vertical -> Connector_PinHeader_2.54mm:PinHeader_1x04_P2.54mm_Vertical
- R_PUP_RES1: value 5K1 -> 200
Connections:
- net +5V: now also J_5V1.2 (Pin_2), LED1.1 (K)
- net GND: now also J_5V1.1 (Pin_1), RL1.1
- net at MCU1.4 (~{RESET}/PB3), SW_RES1.1: now also LED2.1 (K); no longer R_PUP_RES1.2
- net at MCU1.7 (PA6), RTC1.5 (SDA), R_PUP_SDA1.2: now also J_DBG_I2C1.1 (Pin_1)
- net at MCU1.9 (PA4), RTC1.6 (SCL), R_PUP_SCL1.2: now also J_DBG_I2C1.2 (Pin_2)
- new net: LED1.2 (A), RL1.2
- new net: LED2.2 (A), R_PUP_RES1.2
- no-connect marks 10 -> 12
Other:
- moved on the sheet: R_PUP_RES1, SW_RES1
