File: NixieClock.kicad_pcb (KiCad board)
At the start: 2 copper layers, 150 x 50 mm, 110 parts, among them Q1_0 BC807, Q1_1 BC807, Q1_2 BC807, Q1_3 BC807, Q1_4 BC807, Q1_5 BC807, Q1_6 BC807, Q1_7 BC807, Q1_8 BC807, Q1_9 BC807, Q2_0 BC807, Q2_1 BC807, Q2_2 BC807, Q2_3 BC807, Q2_4 BC807, Q2_5 BC807, Q2_6 BC807, Q2_7 BC807, Q2_8 BC807, Q2_9 BC807, Q3_0 BC807, Q3_1 BC807, Q3_2 BC807, Q3_3 BC807, Q3_4 BC807, Q3_5 BC807, Q3_6 BC807, Q3_7 BC807, Q3_8 BC807, Q3_9 BC807, Q4_0 BC807, Q4_1 BC807, Q4_2 BC807, Q4_3 BC807, Q4_4 BC807, Q4_5 BC807, Q4_6 BC807, Q4_7 BC807, Q4_8 BC807, Q4_9 BC807

Commit message: update
Parts:
- removed C1: 1pF, Capacitor_SMD:C_1206_3216Metric_Pad1.33x1.80mm_HandSolder
- removed C2: 2.2pF, Capacitor_SMD:C_1206_3216Metric_Pad1.33x1.80mm_HandSolder
- removed CR2: 10MHz, Crystal:Crystal_SMD_HC49-SD_HandSoldering
- removed F1: 250V/0.5A, NixieClock:Breaker_Holder_5x20
- added J_5V1: Conn_01x02_Pin, Connector_PinHeader_2.54mm:PinHeader_1x02_P2.54mm_Vertical, B.Cu at (150.0, 91.5)
- added J_DBG_I2C1: Conn_01x02_Pin, Connector_PinHeader_2.54mm:PinHeader_1x02_P2.54mm_Vertical, B.Cu at (163.0, 91.0)
- added LED1: LED, LED_SMD:LED_1206_3216Metric_Pad1.42x1.75mm_HandSolder, B.Cu at (57.5, 120.3)
- added LED2: LED, LED_SMD:LED_1206_3216Metric_Pad1.42x1.75mm_HandSolder, B.Cu at (57.5, 125.0)
- added RL1: 200, Resistor_SMD:R_1206_3216Metric_Pad1.30x1.75mm_HandSolder, B.Cu at (57.5, 115.0)
- CR1, MCU1, REG1, RTC1, R_PUP_SCL1, R_PUP_SDA1, SR1, SR2, SR3, SR4, SR5, SW_RES1: moved to B.Cu
- J_12V1: footprint Connector_PinHeader_2.00mm:PinHeader_1x02_P2.00mm_Vertical -> Connector_PinHeader_2.54mm:PinHeader_1x02_P2.54mm_Vertical; moved to B.Cu
- J_170V1: footprint Connector_PinHeader_2.00mm:PinHeader_1x01_P2.00mm_Vertical -> Connector_PinHeader_2.54mm:PinHeader_1x01_P2.54mm_Vertical; moved to B.Cu
- J_BTN1: footprint Connector_PinHeader_2.00mm:PinHeader_1x03_P2.00mm_Vertical -> Connector_PinHeader_2.54mm:PinHeader_1x03_P2.54mm_Vertical; moved to B.Cu
- J_DBG1: footprint Connector_PinHeader_2.00mm:PinHeader_1x04_P2.00mm_Vertical -> Connector_PinHeader_2.54mm:PinHeader_1x04_P2.54mm_Vertical; moved to B.Cu
- R_PUP_RES1: value 5K1 -> 200; moved to B.Cu
- moved BT1 241.2 mm to (-68.0, 27.9), turned to 90 degrees
- moved SW_RES1 203.0 mm to (79.0, -27.0), turned to 180 degrees
- moved CR1 202.9 mm to (72.3, -20.0), turned to 180 degrees
- moved RTC1 202.3 mm to (64.0, -27.0), turned to 180 degrees
- moved R4_7 185.9 mm to (15.0, 6.00), turned to -90 degrees
- moved R4_6 180.0 mm to (20.0, 6.00), turned to -90 degrees
- moved REG1 177.9 mm to (-21.5, 33.8), turned to 90 degrees
- moved R4_4 177.1 mm to (7.00, 17.0), turned to 180 degrees
- moved R4_5 174.3 mm to (25.0, 6.00), turned to -90 degrees
- moved R4_3 171.8 mm to (7.00, 22.0), turned to 180 degrees
- moved R4_2 166.2 mm to (7.00, 28.0), turned to 180 degrees
- moved R3_7 163.6 mm to (45.0, 6.00), turned to -90 degrees
- moved R4_8 162.1 mm to (15.0, 44.0), turned to 90 degrees
- moved SR5 161.4 mm to (7.00, 8.00), turned to 180 degrees
- moved R4_1 161.4 mm to (7.00, 33.0), turned to 180 degrees
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Connections:
- MCU1 pad 2: Net-(MCU1-XTAL1/PB0) -> unconnected-(MCU1-XTAL1/PB0-Pad2)
- MCU1 pad 3: Net-(MCU1-XTAL2/PB1) -> unconnected-(MCU1-XTAL2/PB1-Pad3)
- MCU1 pad 4: Net-(MCU1-~{RESET}/PB3) -> Net-(LED2-K)
- R_PUP_RES1 pad 2: Net-(MCU1-~{RESET}/PB3) -> Net-(LED2-A)
- SW_RES1 pad 1: Net-(MCU1-~{RESET}/PB3) -> Net-(LED2-K)
Routing:
- net /+170V: track 0.00 -> 101.3 mm, vias 0 -> 4
- net Net-(Q4_3-B): track 0.00 -> 81.3 mm
- net Net-(Q1_9-B): track 0.00 -> 81.2 mm
- net Net-(Q1_8-B): track 0.00 -> 79.3 mm
- net Net-(Q4_2-B): track 0.00 -> 78.7 mm
- net Net-(SR1-QP1): track 0.00 -> 65.9 mm, vias 0 -> 1
- net Net-(Q4_4-B): track 0.00 -> 65.4 mm
- net Net-(Q1_0-B): track 0.00 -> 65.3 mm
- net Net-(Q4_1-B): track 0.00 -> 63.3 mm
- net Net-(Q1_7-B): track 0.00 -> 63.3 mm
- net Net-(SR1-QP2): track 0.00 -> 58.2 mm, vias 0 -> 1
- net Net-(SR1-QP3): track 0.00 -> 50.5 mm, vias 0 -> 1
- net Net-(SR1-QP0): track 0.00 -> 27.9 mm, vias 0 -> 1
- net Net-(SR2-QP1): track 0.00 -> 26.9 mm, vias 0 -> 1
- net Net-(N4-A): track 0.00 -> 21.5 mm
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
Commit message: pcb update
Routing:
- net Net-(SR4-QP0): track 0.00 -> 103.8 mm
- net /+5V: track 0.00 -> 84.1 mm
- net /STR: track 0.00 -> 83.9 mm
- net Net-(SR2-QP2): track 0.00 -> 80.3 mm
- net Net-(SR3-QP4): track 0.00 -> 71.7 mm
- net Net-(SR3-QP5): track 0.00 -> 70.7 mm
- net Net-(SR3-QP6): track 0.00 -> 65.5 mm
- net Net-(SR3-QP7): track 0.00 -> 59.1 mm
- net Net-(SR2-QP3): track 0.00 -> 57.3 mm
- net Net-(SR4-QP5): track 0.00 -> 56.2 mm
- net Net-(SR4-QP7): track 0.00 -> 55.1 mm
- net Net-(SR2-QP4): track 0.00 -> 54.7 mm
- net Net-(SR5-QP7): track 0.00 -> 52.0 mm
- net Net-(SR4-QP4): track 0.00 -> 51.6 mm
- net Net-(SR4-QP6): track 0.00 -> 48.1 mm
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